Commit message: Add collision code

File: description/caster_wheel.xacro (robot description, xacro)
@@ -11,4 +11,9 @@
             <material name="white" />
         </visual>
+        <collision>
+            <geometry>
+                <sphere radius="0.06" />
+            </geometry>
+        </collision>
     </link>
     <joint name="caster_wheel_joint" type="fixed">

File: description/chassis.xacro (robot description, xacro)
@@ -8,4 +8,9 @@
             </geometry>
         </visual>
+        <collision>
+            <geometry>
+                <box size="0.45 0.3 0.17" />
+            </geometry>
+        </collision>
     </link>
     <joint name="chassis_joint" type="fixed" >

File: description/wheels.xacro (robot description, xacro)
@@ -11,4 +11,9 @@
             <material name="black" />
         </visual>
+        <collision>
+            <geometry>
+                <cylinder radius="0.06" length="0.05" />
+            </geometry>
+        </collision>
     </link>
     <joint name="left_wheel_joint" type="fixed" >
@@ -24,4 +29,9 @@
             <material name="black" />
         </visual>
+        <collision>
+            <geometry>
+                <cylinder radius="0.06" length="0.05" />
+            </geometry>
+        </collision>
     </link>
     <joint name="right_wheel_joint" type="fixed" >

Commit message: Add inertia code for the caster wheel and chassis

File: description/caster_wheel.xacro (robot description, xacro)
@@ -16,4 +16,15 @@
             </geometry>
         </collision>
+        <inertial>
+            <mass value="0.00594" />
+            <inertia
+                ixx="0.0000085536"
+                ixy="0.0"
+                ixz="0.0"
+                iyy="0.0000085536"
+                iyz="0.0"
+                izz="0.0000085536"
+            />
+        </inertial>
     </link>
     <joint name="caster_wheel_joint" type="fixed">

File: description/chassis.xacro (robot description, xacro)
@@ -13,4 +13,15 @@
             </geometry>
         </collision>
+        <inertial>
+            <mass value="0.1518" />
+            <inertia
+                ixx="0.001504085"
+                ixy="0.0"
+                ixz="0.0"
+                iyy="0.00292721 "
+                iyz="0.0"
+                izz="0.003700125"
+            />
+        </inertial>
     </link>
     <joint name="chassis_joint" type="fixed" >
