Commit message: Add code to move the back wheels further out so that they do not overlap with the chassis

File: description/back_wheels.xacro (robot description, xacro)
@@ -31,5 +31,5 @@
         <parent link="base_link" />
         <child link="left_wheel_link" />
-        <origin xyz="-0.1125 0.15 -0.085" rpy="-${pi/2} 0 0" />
+        <origin xyz="-0.1125 0.2 -0.085" rpy="-${pi/2} 0 0" />
         <axis xyz="0 0 1" />
     </joint>
@@ -61,5 +61,5 @@
         <parent link="base_link" />
         <child link="right_wheel_link" />
-        <origin xyz="-0.1125 -0.15 -0.085" rpy="${pi/2} 0 0" />
+        <origin xyz="-0.1125 -0.2 -0.085" rpy="${pi/2} 0 0" />
         <axis xyz="0 0 -1" />
     </joint>
@@ -70,5 +70,5 @@
             <right_joint>right_wheel_joint</right_joint>
             <!-- Sets specific wheel measurements -->
-            <wheel_separation>0.225</wheel_separation>
+            <wheel_separation>0.4</wheel_separation>
             <wheel_radius>0.06</wheel_radius>
             <max_linear_acceleration>0.4</max_linear_acceleration>
